File: fuente_317_337/fuente_317_337.kicad_pcb (KiCad board)
At the start: 2 copper layers, 80 x 61 mm, 52 parts, among them J1 Fuente, J10 SEL_7905, J11 -5, J12 ADC+, J13 ADC-, J2 Salida, J3 Salida_12v, J4 Cooler, J5 +5, J6 GND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

Commit message: finish tp8
Parts:
- U4: value LM317_TO-220 -> LM317
Other:
- board text added: "Pablo Gomez - 2024"
- board text removed: "Pablo Gomez DAC - 2024"
Changed lines of the file:
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@@
 			(at 0 -2.33 0)
 			(layer "F.SilkS")
+			(hide yes)
 			(effects
 				(font
@@
 		)
 		(property "Value" "Cooler"
-			(at 0 4.87 0)
+			(at 4.96 4.51 0)
 			(layer "F.Fab")
 			(effects
@@
 		(tags "LED diameter 5.0mm 2 pins")
 		(property "Reference" "D5"
-			(at 1.27 -3.96 0)
+			(at 3.7 3.95 0)
 			(layer "F.SilkS")
 			(effects
@@
 		)
 		(property "Value" "10uF"
-			(at 1.25 3.75 90)
+			(at 1.3 -5.25 -90)
 			(layer "F.Fab")
 			(effects
@@
 		)
 		(fp_text user "${REFERENCE}"
-			(at 1.25 0 90)
+			(at 1.25 -4 -90)
 			(layer "F.Fab")
 			(effects
@@
 		)
 		(property "Value" "E330"
-			(at 15.24 4.32 0)
+			(at 15.245 0 0)
 			(layer "F.Fab")
 			(effects
@@
 		(tags "Diode DO-41_SOD81 series Axial Horizontal pin pitch 10.16mm  length 5.2mm diameter 2.7mm")
 		(property "Reference" "D7"
-			(at 5.08 -2.47 360)
+			(at 5.08 -2.47 0)
 			(layer "F.SilkS")
 			(effects
@@
 		)
 		(property "Value" "1N4007"
-			(at 5.08 2.47 360)
+			(at 5.08 2.47 0)
 			(layer "F.Fab")
 			(effects
@@
 		)
 		(fp_text user "K"
-			(at 0 -2.1 360)
+			(at 0 -2.1 0)
 			(layer "F.SilkS")
 			(effects
@@
 		)
 		(fp_text user "${REFERENCE}"
-			(at 5.47 0 360)
+			(at 5.47 0 0)
 			(layer "F.Fab")
 			(effects
@@
 		)
 		(fp_text user "K"
-			(at 0 -2.1 360)
+			(at 0 -2.1 0)
 			(layer "F.Fab")
 			(effects
@@
 		(tags "mounting hole 3.2mm no annular m3")
 		(property "Reference" "H3"
-			(at 0 -4.2 0)
+			(at 2.28 3.82 0)
 			(layer "F.SilkS")
 			(effects
@@
 			(at 0 4.2 0)
 			(layer "F.Fab")
+			(hide yes)
 			(effects
 				(font
@@
 		)
 		(property "Value" "MountingHole"
-			(at 0 4.2 0)
+			(at 1.64 4.32 0)
 			(layer "F.Fab")
 			(effects
@@
 			)
 		)
-		(property "Value" "LM317_TO-220"
-			(at 2.54 2.5 0)
+		(property "Value" "LM317"
+			(at 5.55 2.405 0)
 			(layer "F.Fab")
 			(effects
@@
 		)
 		(property "Value" "1N4007"
-			(at 5.08 2.47 0)
+			(at 1.65 2.6 0)
 			(layer "F.Fab")
 			(effects
@@
 		)
 		(property "Value" "Cooler"
-			(at 0 4.87 90)
+			(at 2.5 1.135 180)
 			(layer "F.Fab")
+			(hide yes)
 			(effects
 				(font
@@
 		(tags "CP Radial series Radial pin pitch 2.50mm  diameter 5mm Electrolytic Capacitor")
 		(property "Reference" "C11"
-			(at 1.25 -3.75 90)
+			(at -2.3 0.075 180)
 			(layer "F.SilkS")
 			(effects
@@
 		)
 		(property "Value" "1uF"
-			(at 1.25 3.75 90)
+			(at -3.75 0.075 180)
 			(layer "F.Fab")
 			(effects
@@
 		(tags "Through hole pin header THT 1x03 2.54mm single row")
 		(property "Reference" "Radj_fino1"
-			(at 0 -2.33 0)
+			(at 2.8 2.55 -90)
 			(layer "F.SilkS")
 			(effects
@@
 		)
 		(property "Value" "510"
-			(at 1.27 2.37 0)
+			(at 1.1 2.65 0)
 			(layer "F.Fab")
 			(effects
@@
 		(layer "Edge.Cuts")
 	)
-	(gr_text "Pablo Gomez\nDAC - 2024"
-		(at 85.65 21.35 0)
+	(gr_text "Pablo Gomez - 2024\n\n"
+		(at 101 21.9 90)
 		(layer "B.Cu")
 		(effects

Commit message: feat: version final para el tp integrador
Parts:
- removed U8: LM385, Package_TO_SOT_THT:TO-92_Inline
- added U1: LM385BZ-1.2, Package_TO_SOT_THT:TO-92_Inline, F.Cu at (46.7, 55.2)
- R1, R2: value 8k1 -> 10k
- U4: value LM317 -> LM317_TO-220
- U7: value LM385 -> LM385BZ-1.2
- moved U7 2.48 mm to (60.5, 31.4), turned to 180 degrees
- moved C10 0.95 mm to (77.3, 53.2)
- moved Radj_fino2 0.29 mm to (70.7, 55.0)
Connections:
- U7 pad 1: GND -> (no net)
- U7 pad 2: GND -> +1V2
- U7 pad 3: +1V2 -> GND
Routing:
- net GND: track 362.6 -> 355.3 mm
- net -1V2: track 15.0 -> 20.1 mm
- net +1V2: track 16.1 -> 13.1 mm
- net +12V: track 158.9 -> 156.9 mm
- net Net-(U5-ADJ): track 20.9 -> 21.7 mm
- net -12V: track 170.5 -> 169.8 mm
