File: fuente_317_esp_8266/fuente_317_esp_8266.kicad_pcb (KiCad board)
At the start: 2 copper layers, 75 x 60 mm, 35 parts, among them J1 UART, J10 Alimentacion, J12 Vadj+, J13 Vadj-, J2 LCD16x2, J3 Vadj+, J4 Vadj-, J5 Vadj+, J6 Vadj-, J8 BTN_MODE, J9 BTN_SEL, U2 CD4051B, U3 LM324, U4 AMS1117-3.3

Commit message: feat: version final para el tp integrador
Parts:
- removed C1, C2: 10uF, Capacitor_THT:CP_Radial_D5.0mm_P2.50mm
- removed D1: LED, LED_THT:LED_D5.0mm
- removed H1, H2, H3, H4: MountingHole, MountingHole:MountingHole_3.2mm_M3
- removed J1: UART, Connector_PinHeader_2.54mm:PinHeader_1x02_P2.54mm_Vertical
- removed J10: Alimentacion, TerminalBlock_Phoenix:TerminalBlock_Phoenix_MKDS-1,5-2-5.08_1x02_P5.08mm_Horizontal
- removed J12, J3, J5: Vadj+, Connector_PinHeader_2.54mm:PinHeader_1x02_P2.54mm_Vertical
- removed J13, J4, J6: Vadj-, Connector_PinHeader_2.54mm:PinHeader_1x02_P2.54mm_Vertical
- removed J2: LCD16x2, Connector_PinHeader_2.54mm:PinHeader_1x04_P2.54mm_Vertical
- removed J8: BTN_MODE, Connector_PinHeader_2.54mm:PinHeader_1x03_P2.54mm_Vertical
- removed J9: BTN_SEL, Connector_PinHeader_2.54mm:PinHeader_1x03_P2.54mm_Vertical
- removed R1, R12, R2, R3, R4, R9: 10k, Resistor_THT:R_Axial_DIN0207_L6.3mm_D2.5mm_P10.16mm_Horizontal
- removed R10, R11, R5, R6, R7: 10k, Resistor_THT:R_Axial_DIN0207_L6.3mm_D2.5mm_P5.08mm_Vertical
- removed R13: 120, Resistor_THT:R_Axial_DIN0207_L6.3mm_D2.5mm_P10.16mm_Horizontal
- removed R8: 47k, Resistor_THT:R_Axial_DIN0207_L6.3mm_D2.5mm_P5.08mm_Vertical
- removed U1: ~, Componentes_Proyecto_Digitales:Esp-8266-DevKit
- removed U2: CD4051B, Package_DIP:CERDIP-16_W7.62mm_SideBrazed_Socket
- removed U3: LM324, Package_DIP:CERDIP-14_W7.62mm_SideBrazed_Socket
- removed U4: AMS1117-3.3, Package_TO_SOT_SMD:SOT-223-3_TabPin2
Routing:
- net GND: track 350.1 -> 0.00 mm
- net +5V: track 146.3 -> 0.00 mm
- net Iadc+: track 90.3 -> 0.00 mm
- net Vadc+: track 77.2 -> 0.00 mm
- net Iadc-: track 57.5 -> 0.00 mm
- net Vadc-: track 56.4 -> 0.00 mm
- net +3V3: track 52.3 -> 0.00 mm
- net Vadc: track 29.5 -> 0.00 mm
- net Vout-: track 24.4 -> 0.00 mm
- net A_mux: track 23.6 -> 0.00 mm
- net B_mux: track 20.5 -> 0.00 mm
- net I2C - SCL: track 18.4 -> 0.00 mm
- net I2C - SDA: track 18.3 -> 0.00 mm
- net BTN_SELECT: track 16.8 -> 0.00 mm
- net Vout+: track 16.3 -> 0.00 mm
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- removed copper zone on B.Cu, net GND
Other:
- board outline removed
- board text removed: "Pablo Gomez DAC 2024 Fuente partida 317 - 337"
